Commit message: adding control to robot

File: diff_bot/urdf/caster_wheel.xacro (robot description, xacro)
@@ -22,5 +22,5 @@
     <!-- Caster Wheel Joit -->
     <joint name="front_caster_wheel_joint" type="fixed">
-        <origin xyz="${caster_wheel_offset_x} 0.0 ${caster_wheel_offset_z}" rpy="0.0 0.0 0.0"/>
+        <origin xyz="0.3 0.0 ${caster_wheel_offset_z}" rpy="0.0 0.0 0.0"/>
         <parent link="chassis_link"/>
         <child link="front_caster_wheel_link"/>
@@ -47,5 +47,5 @@
     <!-- Caster Wheel Joit -->
     <joint name="back_caster_wheel_joint" type="fixed">
-        <origin xyz="${back_caster_wheel_offset_x} 0.0 ${caster_wheel_offset_z}" rpy="0.0 0.0 0.0"/>
+        <origin xyz="0.01 0.0 ${caster_wheel_offset_z}" rpy="0.0 0.0 0.0"/>
         <parent link="chassis_link"/>
         <child link="back_caster_wheel_link"/>
@@ -61,5 +61,5 @@
     </link>
     <joint name="holder_joint" type="fixed">
-        <origin xyz="${caster_wheel_offset_x} 0.0 0.0" rpy="0.0 0.0 0.0"/>
+        <origin xyz="0.30 0.0 0.0" rpy="0.0 0.0 0.0"/>
         <parent link="chassis_link"/>
         <child link="caster_holder"/>
@@ -74,11 +74,17 @@
     </link>
     <joint name="back_holder_joint" type="fixed">
-        <origin xyz="${back_caster_wheel_offset_x} 0.0 0.0" rpy="0.0 0.0 0.0"/>
+        <origin xyz="0.01 0.0 0.0" rpy="0.0 0.0 0.0"/>
         <parent link="chassis_link"/>
         <child link="back_caster_holder"/>
     </joint>
-    <gazebo reference="caster_wheel_link">
+    <gazebo reference="front_caster_wheel_link">
         <mu1 value="0.001"/>
         <mu2 value="0.001"/>
+        <material> Gazebo/Green </material>
+    </gazebo>
+    <gazebo reference="back_caster_wheel_link">
+        <mu1 value="0.001"/>
+        <mu2 value="0.001"/>
+        <material> Gazebo/Red </material>
     </gazebo>
 </robot>

File: diff_bot/urdf/chassis.xacro (robot description, xacro)
@@ -7,9 +7,9 @@
                 <cylinder radius="${chassis_length}" length="${chassis_height}"/>
             </geometry>
-            <origin xyz="${chassis_length/2} 0.0 ${chassis_height/2}"/>
+            <origin xyz="0.155 0.0 ${chassis_height/2}"/>
             <material name="green"/>
         </visual>
         <collision>
-            <origin xyz="${chassis_length/2} 0.0 ${chassis_height/2}"/>
+            <origin xyz="0.155 0.0 ${chassis_height/2}"/>
         </collision>
         <xacro:inertial_box mass="${chassis_mass}" x="${chassis_length}" y="${chassis_width}" z="${chassis_height}">
@@ -21,5 +21,5 @@
         <parent link="base_link"/>
         <child link="chassis_link"/>
-        <origin xyz="-${wheel_offset_x} 0.0 0.0"/>
+        <origin xyz="-0.155 0.0 0.0"/>
     </joint>
     <gazebo reference="chassis_link">

File: diff_bot/urdf/control.xacro (robot description, xacro)
@@ -10,5 +10,5 @@
                 <param name="baud_rate">57600</param>
                 <param name="timeout">1000</param>
-                <param name="enc_counts_per_rev">1500</param>
+                <param name="enc_counts_per_rev">897</param>
         </hardware>
         <joint name="left_wheel_joint">

File: diff_bot/urdf/gazebo_control.xacro (robot description, xacro)
@@ -6,6 +6,6 @@
             <left_joint>left_wheel_joint</left_joint>
             <right_joint>right_wheel_joint</right_joint>
-            <wheel_separation>0.24</wheel_separation>
-            <wheel_diameter>0.065</wheel_diameter>
+            <wheel_separation>0.225</wheel_separation>
+            <wheel_diameter>0.07</wheel_diameter>
             <!-- Limits-->
             <max_wheel_torque>200</max_wheel_torque>

File: diff_bot/urdf/lidar.xacro (robot description, xacro)
@@ -16,5 +16,5 @@
     </gazebo>
     <joint name="laser_joint" type="fixed">
-        <origin xyz="0.07 0.0 0.18" rpy="0.0 0.0 0.0"/>
+        <origin xyz="0.155 0.0 0.18" rpy="0.0 0.0 0.0"/>
         <parent link="chassis_link"/>
         <child link="laser_frame"/>

File: diff_bot/urdf/properties.xacro (robot description, xacro)
@@ -19,5 +19,5 @@
     <xacro:property name="caster_wheel_offset_x" value="0.22"/>
     <xacro:property name="back_caster_wheel_offset_x" value="-0.06"/>
-    <xacro:property name="caster_wheel_offset_z" value="-0.0255"/>
+    <xacro:property name="caster_wheel_offset_z" value="-0.0258"/>
                                 <!-- Colors -->
     <material name="white">

File: diff_bot/urdf/wheels.xacro (robot description, xacro)
@@ -23,5 +23,5 @@
     <xacro:macro name="wheel_joint" params="joint_name wheel_name y_offset ">
         <joint name="${joint_name}" type="continuous">
-            <origin xyz="0.038 ${y_offset} 0" rpy="${-pi/2} 0.0 0.0"/>
+            <origin xyz="0.0 ${y_offset} 0" rpy="${-pi/2} 0.0 0.0"/>
             <parent link="base_link"/>
             <child link="${wheel_name}"/>
@@ -37,9 +37,31 @@
     <!-- Right Wheel Joint -->
     <xacro:wheel_joint joint_name="right_wheel_joint" wheel_name="right_wheel_link" y_offset="${-wheel_offset_y}"/>
-    <gazebo reference="left_wheel_link">
+    <!-- <gazebo reference="left_wheel_link">
         <material> Gazebo/Black </material>
     </gazebo>
     <gazebo reference="right_wheel_link">
         <material> Gazebo/Black </material>
+    </gazebo> -->
+    <gazebo reference="left_wheel_link">
+        <material> Gazebo/Black </material>
+        <mu1>0.9</mu1>
+        <mu2>0.9</mu2>
+      <minDepth>0.001</minDepth>
+        <kp>100000000</kp>
+        <kd>1</kd>
     </gazebo>
+    <gazebo reference="right_wheel_link">
+        <material> Gazebo/Black </material>
+        <mu1>0.9</mu1>
+        <mu2>0.9</mu2>
+      <minDepth>0.001</minDepth>
+        <kp>100000000</kp>
+        <kd>1</kd>
+    </gazebo>
+    <gazebo reference="left_wheel_hinge">
+        <implicitSpringDamper>true</implicitSpringDamper>
+ </gazebo>
+ <gazebo reference="right_wheel_hinge">
+        <implicitSpringDamper>true</implicitSpringDamper>
+ </gazebo>
 </robot>
