Commit message: nav done

File: diff_bot/urdf/chassis.xacro (robot description, xacro)
@@ -11,4 +11,7 @@
         </visual>
         <collision>
+            <geometry>
+                <cylinder radius="${chassis_length}" length="${chassis_height}"/>
+            </geometry>
             <origin xyz="0.155 0.0 ${chassis_height/2}"/>
         </collision>
@@ -24,5 +27,5 @@
     </joint>
     <gazebo reference="chassis_link">
-        <material> Gazebo/Grey </material>
+        <material> Gazebo/Red </material>
     </gazebo>
 </robot>
